File: hardware/colony/Colony.brd (EAGLE design)
At the start: 25.3 x 26 mm, 56 parts, among them IC1 MSP430FR5728, IC2 nRF24AP2-1CH, IC3 LM75, J4 SL127L6TH, Q1 16 MHz, Q2 32 kHz, Q3 32 kHz, U1 TPS61097-33DBVT

Commit message: Connected nRF24AP2-1CH pad to GND.
Routing:
- net GND: vias 49 -> 53
Changed lines of the file:
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@@
 <?xml version="1.0" encoding="utf-8"?>
 <!DOCTYPE eagle SYSTEM "eagle.dtd">
-<eagle version="6.2">
+<eagle version="6.4">
 <drawing>
 <settings>
@@
 </class>
 </classes>
-<designrules>
+<designrules name="default">
 <description language="de">&lt;b&gt;EAGLE Design Rules&lt;/b&gt;
 &lt;p&gt;
@@
 <wire x1="1.524" y1="5.588" x2="0.9652" y2="5.588" width="0.254" layer="1"/>
 <wire x1="0.9652" y1="5.588" x2="0.4572" y2="6.096" width="0.254" layer="1"/>
+<via x="13.335" y="16.637" extent="1-16" drill="0.3048" alwaysstop="yes"/>
+<via x="14.859" y="16.637" extent="1-16" drill="0.3048" alwaysstop="yes"/>
+<via x="14.859" y="15.113" extent="1-16" drill="0.3048" alwaysstop="yes"/>
+<via x="14.097" y="15.875" extent="1-16" drill="0.3048" alwaysstop="yes"/>
 </signal>
 <signal name="N$4">
@@
 </signal>
 </signals>
-<errors>
-</errors>
 </board>
 </drawing>
